Commit message: Add MoveIt C++ node, update URDF, integrate ros2_control and fix configs

File: src/my_robot_description/urdf/arm.xacro (robot description, xacro)
@@ -1,4 +1,10 @@
 <?xml version="1.0"?>
 <robot xmlns:xacro="http://www.ros.org/wiki/xacro">
+    <link name="world"/>
+    <joint name="world_joint" type="fixed">
+        <parent link="world"/>
+        <child link="base_link"/>
+        <origin xyz="0 0 0" rpy="0 0 0"/>
+    </joint>
     <link name="base_link">
         <visual>
@@ -9,4 +15,6 @@
             <material name="grey" />
         </visual>
+       <xacro:box_inertia m="5.0" x="0.4" y="0.4" z="0.1"
+                           o_xyz="0 0 0.05" o_rpy="0 0 0" />
         <collision>
             <geometry>
@@ -30,4 +38,6 @@
             <origin xyz="0 0 0.25" rpy="0 0 0" />
         </collision>
+       <xacro:box_inertia m="5.0" x="0.2" y="0.2" z="0.5"
+                           o_xyz="0 0 0.25" o_rpy="0 0 0" />
     </link>
     <link name="arm_link">
@@ -45,4 +55,6 @@
             <origin xyz="0 0 0.3" rpy="0 0 0" />
         </collision>
+        <xacro:box_inertia m="5.0" x="0.1" y="0.1" z="0.6"
+                           o_xyz="0 0 0.3" o_rpy="0 0 0" />
     </link>
     <link name="elbow_link">
@@ -60,4 +72,6 @@
             <origin xyz="0 0 0.05" rpy="0 0 0" />
         </collision>
+          <xacro:box_inertia m="5.0" x="0.1" y="0.1" z="0.1"
+                           o_xyz="0 0 0.05" o_rpy="0 0 0" />
     </link>
     <link name="forearm_link">
@@ -75,4 +89,6 @@
             <origin xyz="0 0 0.25" rpy="0 0 0" />
         </collision>
+        <xacro:box_inertia m="5.0" x="0.1" y="0.1" z="0.5"
+                           o_xyz="0 0 0.25" o_rpy="0 0 0" />
     </link>
     <link name="wrist_link">
@@ -90,4 +106,6 @@
             <origin xyz="0 0 0.025" rpy="0 0 0" />
         </collision>
+          <xacro:box_inertia m="5.0" x="0.1" y="0.1" z="0.05"
+                           o_xyz="0 0 0.05" o_rpy="0 0 0" />
     </link>
     <link name="hand_link">
@@ -105,4 +123,6 @@
             <origin xyz="0 0 0.01" rpy="0 0 0" />
         </collision>
+        <xacro:box_inertia m="5.0" x="0.1" y="0.1" z="0.02"
+                           o_xyz="0 0 0.01" o_rpy="0 0 0" />
     </link>
     <link name="tool_link" />
@@ -155,2 +175,91 @@
     </joint>
 </robot>
+    <!-- ==================== GAZEBO PLUGINS ==================== -->
+    <!-- 1. GAZEBO PHYSICS & CONTACT PROPERTIES -->
+    <!-- <gazebo>
+        <physics name="default_physics" default="true" type="ode">
+            <max_step_size>0.001</max_step_size>
+            <real_time_factor>1.0</real_time_factor>
+            <real_time_update_rate>1000</real_time_update_rate>
+            <gravity>0 0 -9.81</gravity>
+            <ode>
+                <solver>
+                    <type>quick</type>
+                    <iters>150</iters>
+                    <precon_iters>0</precon_iters>
+                    <sor>1.400000</sor>
+                    <use_dynamic_moi_rescaling>0</use_dynamic_moi_rescaling>
+                </solver>
+                <constraints>
+                    <cfm>0.00000</cfm>
+                    <erp>0.20000</erp>
+                    <contact_max_correcting_vel>2000.00000</contact_max_correcting_vel>
+                    <contact_surface_layer>0.01000</contact_surface_layer>
+                </constraints>
+            </ode>
+        </physics>
+    </gazebo>
+    <!- 2. LINK SURFACE PROPERTIES (Friction, Bounce) -->
+    <!-- <gazebo reference="base_link">
+        <material>Gazebo/Grey</material>
+        <mu1>0.8</mu1>
+        <mu2>0.8</mu2>
+        <kp>1000000.0</kp>
+        <kd>1.0</kd>
+    </gazebo>
+    <gazebo reference="shoulder_link">
+        <material>Gazebo/Blue</material>
+        <mu1>0.8</mu1>
+        <mu2>0.8</mu2>
+    </gazebo>
+    <gazebo reference="arm_link">
+        <material>Gazebo/Grey</material>
+        <mu1>0.8</mu1>
+        <mu2>0.8</mu2>
+    </gazebo>
+    <gazebo reference="elbow_link">
+        <material>Gazebo/Blue</material>
+        <mu1>0.8</mu1>
+        <mu2>0.8</mu2>
+    </gazebo>
+    <gazebo reference="forearm_link">
+        <material>Gazebo/Grey</material>
+        <mu1>0.8</mu1>
+        <mu2>0.8</mu2>
+    </gazebo>
+    <gazebo reference="wrist_link">
+        <material>Gazebo/Blue</material>
+        <mu1>0.8</mu1>
+        <mu2>0.8</mu2>
+    </gazebo>
+    <gazebo reference="hand_link">
+        <material>Gazebo/Grey</material>
+        <mu1>0.8</mu1>
+        <mu2>0.8</mu2>
+    </gazebo>
+    <!- 3. JOINT FRICTION & DAMPING -->
+    <!-- <gazebo reference="joint1">
+        <implicitSpringDamper>1</implicitSpringDamper>
+        <friction>0.0</friction>
+    </gazebo>
+    <gazebo reference="joint2">
+        <implicitSpringDamper>1</implicitSpringDamper>
+        <friction>0.0</friction>
+    </gazebo>
+    <gazebo reference="joint3">
+        <implicitSpringDamper>1</implicitSpringDamper>
+        <friction>0.0</friction>
+    </gazebo>
+    <gazebo reference="joint4">
+        <implicitSpringDamper>1</implicitSpringDamper>
+        <friction>0.0</friction>
+    </gazebo>
+    <gazebo reference="joint5">
+        <implicitSpringDamper>1</implicitSpringDamper>
+        <friction>0.0</friction>
+    </gazebo>
+    <gazebo reference="joint6">
+        <implicitSpringDamper>1</implicitSpringDamper>
+        <friction>0.0</friction>
+    </gazebo> -->
+ <!-- -->

File: src/my_robot_description/urdf/common_properties.xacro (robot description, xacro)
@@ -13,3 +13,21 @@
         <color rgba="0 0.6 0 1"/>
     </material>
+     <xacro:macro name="box_inertia" params="m x y z o_xyz o_rpy">
+        <inertial>
+            <mass value="${m}" />
+            <origin xyz="${o_xyz}" rpy="${o_rpy}" />
+            <inertia ixx="${(m/12) * (y*y + z*z)}" ixy="0" ixz="0"
+                     iyy="${(m/12) * (x*x + z*z)}" iyz="0"
+                     izz="${(m/12) * (x*x + y*y)}" />
+        </inertial>
+    </xacro:macro>
+    <!-- <xacro:macro name="cylinder_inertia" params="m r l o_xyz o_rpy">
+        <inertial>
+            <mass value="${m}" />
+            <origin xyz="${o_xyz}" rpy="${o_rpy}" />
+            <inertia ixx="${(m/12) * (3*r*r + l*l)}" ixy="0" ixz="0"
+                     iyy="${(m/12) * (3*r*r + l*l)}" iyz="0"
+                     izz="${(m/2) * (r*r)}" />
+        </inertial>
+    </xacro:macro> -->
 </robot>

File: src/my_robot_description/urdf/gripper.xacro (robot description, xacro)
@@ -15,4 +15,6 @@
                  <origin xyz="0 0 0.01" rpy="0 0 0" />
             </collision>
+             <xacro:box_inertia m="1.0" x="0.2" y="0.06" z="0.02"
+                           o_xyz="0 0 0.01" o_rpy="0 0 0" />
         </link>
         <link name="gripper_left_finger_link">
@@ -30,4 +32,6 @@
             <origin xyz="0 0 0.04" rpy="0 0 0" />
         </collision>
+         <xacro:box_inertia m="1.0" x="0.02" y="0.06" z="0.08"
+                           o_xyz="0 0 0.0" o_rpy="0 0 0" />
     </link>
     <link name="gripper_right_finger_link">
@@ -45,4 +49,6 @@
             <origin xyz="0 0 0.04" rpy="0 0 0" />
         </collision>
+         <xacro:box_inertia m="1.0" x="0.02" y="0.06" z="0.08"
+                           o_xyz="0 0 0.0" o_rpy="0 0 0" />
     </link>
     <joint name="gripper_left_finger_joint" type="prismatic">

File: src/my_robot_description/urdf/my_robot_urdf.xacro (robot description, xacro)
@@ -4,5 +4,12 @@
     <xacro:include filename="arm.xacro"/>
     <xacro:include filename="gripper.xacro"/>
-    <xacro:include filename="my_robot_ros2_control.xacro"/>
+    <xacro:include filename="my_robot.ros2_control.xacro"/>
+  <!-- THIS LINE IS CRITICAL -->
+    <!-- <gazebo>
+        <plugin filename="gz_ros2_control-system"
+                name="gz_ros2_control::GazeboSimROS2ControlPlugin">
+        <parameters>$(find my_robot_bringup)/config/ros2_controllers.yaml</parameters>
+        </plugin>
+    </gazebo> -->
     <joint name="base_to_arm_joint" type="fixed">
         <parent link="tool_link"/>

Commit message: Add MoveIt2 pick and place pipeline with gripper control

File: src/my_robot_description/urdf/arm.xacro (robot description, xacro)
@@ -126,5 +126,27 @@
                            o_xyz="0 0 0.01" o_rpy="0 0 0" />
     </link>
-    <link name="tool_link" />
+    <link name="camera_link">
+        <visual>
+            <geometry>
+                <box size="0.1 0.1 0.02"/>
+            </geometry>
+            <origin xyz="0 0 0" rpy="0 0 0" />
+            <material name="grey"/>
+        </visual>
+        <collision>
+            <geometry>
+                <box size="0.1 0.1 0.02"/>
+            </geometry>
+             <origin xyz="0 0 0" rpy="0 0 0"/>
+        </collision>
+        <xacro:box_inertia m="0.1" x="0.1" y="0.1" z="0.02"
+                           o_xyz="0 0 0" o_rpy="0 0 0" />
+    </link>
+    <link name="tool_link" >
+        <inertial>
+            <mass value="0.01"/>
+            <inertia ixx="0.000001" ixy="0.0" ixz="0.0" iyy="0.000001" iyz="0.0" izz="0.000001"/>
+        </inertial>
+    </link>
     <joint name="joint1" type="revolute">
         <parent link="base_link" />
@@ -174,92 +196,41 @@
         <origin xyz="0 0 0.02" rpy="0 0 0" />
     </joint>
+    <joint name="world_to_camera_joint" type="fixed">
+        <parent link="world"/>
+        <child link="camera_link"/>
+        <origin xyz="0.5 0.5 2.0" rpy="0 1.57 0"/>
+    </joint>
+    <joint name="camera_optical_joint" type="fixed">
+        <parent link="camera_link"/>
+        <child link="camera_link_optical"/>
+        <origin xyz="0 0 0" rpy="0 1.57 0"/>
+    </joint>
+    <link name="camera_link_optical">
+        <inertial>
+            <mass value="0.001"/>
+            <inertia ixx="0.0000001" ixy="0.0" ixz="0.0" iyy="0.0000001" iyz="0.0" izz="0.0000001"/>
+        </inertial>
+    </link>
+    <gazebo reference="camera_link">
+            <sensor name="camera" type="camera">
+                <camera>
+                    <horizontal_fov>1.047</horizontal_fov>
+                    <image>
+                        <width>640</width>
+                        <height>480</height>
+                        <format>R8G8B8</format>
+                    </image>
+                    <clip>
+                        <near>0.1</near>
+                        <far>20</far>
+                    </clip>
+                <optical_frame_id>camera_link_optical</optical_frame_id>
+                <camera_info_topic>camera/camera_info</camera_info_topic>
+            </camera>
+            <always_on>1</always_on>
+            <update_rate>20</update_rate>
+            <visualize>true</visualize>
+            <topic>camera/image_raw</topic>
+        </sensor>
+    </gazebo>
 </robot>
-    <!-- ==================== GAZEBO PLUGINS ==================== -->
-    <!-- 1. GAZEBO PHYSICS & CONTACT PROPERTIES -->
-    <!-- <gazebo>
-        <physics name="default_physics" default="true" type="ode">
-            <max_step_size>0.001</max_step_size>
-            <real_time_factor>1.0</real_time_factor>
-            <real_time_update_rate>1000</real_time_update_rate>
-            <gravity>0 0 -9.81</gravity>
-            <ode>
-                <solver>
-                    <type>quick</type>
-                    <iters>150</iters>
-                    <precon_iters>0</precon_iters>
-                    <sor>1.400000</sor>
-                    <use_dynamic_moi_rescaling>0</use_dynamic_moi_rescaling>
-                </solver>
-                <constraints>
-                    <cfm>0.00000</cfm>
-                    <erp>0.20000</erp>
-                    <contact_max_correcting_vel>2000.00000</contact_max_correcting_vel>
-                    <contact_surface_layer>0.01000</contact_surface_layer>
-                </constraints>
-            </ode>
-        </physics>
-    </gazebo>
-    <!- 2. LINK SURFACE PROPERTIES (Friction, Bounce) -->
-    <!-- <gazebo reference="base_link">
-        <material>Gazebo/Grey</material>
-        <mu1>0.8</mu1>
-        <mu2>0.8</mu2>
-        <kp>1000000.0</kp>
-        <kd>1.0</kd>
-    </gazebo>
-    <gazebo reference="shoulder_link">
-        <material>Gazebo/Blue</material>
-        <mu1>0.8</mu1>
-        <mu2>0.8</mu2>
-    </gazebo>
-    <gazebo reference="arm_link">
-        <material>Gazebo/Grey</material>
-        <mu1>0.8</mu1>
-        <mu2>0.8</mu2>
-    </gazebo>
-    <gazebo reference="elbow_link">
-        <material>Gazebo/Blue</material>
-        <mu1>0.8</mu1>
-        <mu2>0.8</mu2>
-    </gazebo>
-    <gazebo reference="forearm_link">
-        <material>Gazebo/Grey</material>
-        <mu1>0.8</mu1>
-        <mu2>0.8</mu2>
-    </gazebo>
-    <gazebo reference="wrist_link">
-        <material>Gazebo/Blue</material>
-        <mu1>0.8</mu1>
-        <mu2>0.8</mu2>
-    </gazebo>
-    <gazebo reference="hand_link">
-        <material>Gazebo/Grey</material>
-        <mu1>0.8</mu1>
-        <mu2>0.8</mu2>
-    </gazebo>
-    <!- 3. JOINT FRICTION & DAMPING -->
-    <!-- <gazebo reference="joint1">
-        <implicitSpringDamper>1</implicitSpringDamper>
-        <friction>0.0</friction>
-    </gazebo>
-    <gazebo reference="joint2">
-        <implicitSpringDamper>1</implicitSpringDamper>
-        <friction>0.0</friction>
-    </gazebo>
-    <gazebo reference="joint3">
-        <implicitSpringDamper>1</implicitSpringDamper>
-        <friction>0.0</friction>
-    </gazebo>
-    <gazebo reference="joint4">
-        <implicitSpringDamper>1</implicitSpringDamper>
-        <friction>0.0</friction>
-    </gazebo>
-    <gazebo reference="joint5">
-        <implicitSpringDamper>1</implicitSpringDamper>
-        <friction>0.0</friction>
-    </gazebo>
-    <gazebo reference="joint6">
-        <implicitSpringDamper>1</implicitSpringDamper>
-        <friction>0.0</friction>
-    </gazebo> -->
- <!-- -->

File: src/my_robot_description/urdf/gripper.xacro (robot description, xacro)
@@ -64,5 +64,5 @@
         <origin xyz="0.07 0 0.02" rpy="0 0 0" />
         <axis xyz="1 0 0" />
-        <mimic joint="gripper_left_finger_joint" multiplier="-1.0" />
+        <!-- <mimic joint="gripper_left_finger_joint" multiplier="-1.0" /> -->
         <limit effort="1000.0" velocity="1.0" lower="-0.06" upper="0.0" />
     </joint>

File: src/my_robot_description/urdf/my_robot.ros2_control.xacro (robot description, xacro)
@@ -4,5 +4,6 @@
       <hardware>
           <!-- By default, set up controllers for simulation. This won't work on real hardware -->
-          <plugin>mock_components/GenericSystem</plugin>
+          <!-- <plugin>mock_components/GenericSystem</plugin> new line -->
+          <plugin>gz_ros2_control/GazeboSimSystem</plugin>
       </hardware>
       <joint name="joint1">
@@ -48,4 +49,10 @@
           </state_interface>
       </joint>
+      <joint name="gripper_right_finger_joint">
+          <command_interface name="position"/>
+          <state_interface name="position">
+            <param name="initial_value">0.0</param>
+          </state_interface>
+      </joint>
   </ros2_control>
 </robot>

File: src/my_robot_description/urdf/my_robot_urdf.xacro (robot description, xacro)
@@ -5,4 +5,5 @@
     <xacro:include filename="gripper.xacro"/>
     <xacro:include filename="my_robot.ros2_control.xacro"/>
+    <xacro:include filename="6axis_robotic_gazebo.xacro"/>
   <!-- THIS LINE IS CRITICAL -->
     <!-- <gazebo>

File: src/my_robot_moveit_config/config/my_robot.ros2_control.xacro (robot description, xacro)
@@ -50,4 +50,10 @@
                 </state_interface>
             </joint>
+            <joint name="gripper_right_finger_joint">
+                <command_interface name="position"/>
+                <state_interface name="position">
+                  <param name="initial_value">${initial_positions['gripper_right_finger_joint']}</param>
+                </state_interface>
+            </joint>
         </ros2_control>
     </xacro:macro>
